File: Arduino_humid/Arduino_humid.kicad_pcb (KiCad board)
At the start: 2 copper layers, 171.5 x 103 mm, 24 parts

Commit message: Fixed .step and added silkscreen lables
Parts:
- renumbered REF** to +5v, REF** to D4, REF** to D5, REF** to D6, REF** to D7, REF** to En, REF** to GND, REF** to LCD_Con, REF** to LED, REF** to LED_B, REF** to LED_G, REF** to LED_R, REF** to P_Off, REF** to P_On, REF** to Power_Off, REF** to Power_On, REF** to R1, REF** to R2, REF** to RESET, REF** to RS, REF** to uINPUT
